File: ControlBreakout.sch (KiCad schematic (older format))
At the start: 42 parts, among them J1 Conn_01x12, J2 Conn_01x12, J3 3v3 Bypass, J4 GND1, J5 GND2, J6 Screw_Terminal_01x02, J7 GND3, Q1 AO3401A, U1 TCA9544A, U2 LP5030, U3 MP2359DJ-LF-Z

Commit message: nearly done on v2
Parts:
- removed U2: LP5030, Package_DFN_QFN:VQFN-46-1EP_5x6mm_P0.4mm_EP2.8x3.8mm, symbol LP5030:LP5030
- added C9: 10uF, Capacitor_SMD:C_0603_1608Metric, symbol Device:C_Small
- added R9: 100K, Resistor_SMD:R_0603_1608Metric, symbol Device:R_Small_US
- added U4: IS32FL3237-TQLA3-TR, Package_QFP:TQFP-48-1EP_7x7mm_P0.5mm_EP5x5mm, symbol IS32FL3237:IS32FL3237-TQLA3-TR
- C3, C5: value 1uF -> 100nF; footprint Capacitor_SMD:C_0402_1005Metric -> Capacitor_SMD:C_0603_1608Metric; LCSC C52923 -> C14663
- C7, C8: footprint Capacitor_SMD:C_0603_1608Metric -> Capacitor_SMD:C_1206_3216Metric
- R1: value 3K -> 3.3K; LCSC C4211 -> C22978
Connections:
- net +3V3: now also C3.1, C9.1, R9.2, U4.39 (SDB), U4.41 (VCC); no longer J2.2 (Pin_2), J2.3 (Pin_3)
- net B1: now also U4.1 (OUT3)
- net B10: now also U4.31 (OUT30)
- net B2: now also U4.5 (OUT6)
- net B3: now also U4.8 (OUT9)
- net B4: now also U4.11 (OUT12)
- net B5: now also U4.14 (OUT15)
- net B6: now also U4.17 (OUT18)
- net B7: now also U4.22 (OUT21)
- net B8: now also U4.25 (OUT24)
- net B9: now also U4.28 (OUT27)
- net G1: now also U4.48 (OUT2)
- net G10: now also U4.30 (OUT29)
- net G2: now also U4.3 (OUT5)
- net G3: now also U4.7 (OUT8)
- net G4: now also U4.10 (OUT11)
- net G5: now also U4.13 (OUT14)
- net G6: now also U4.16 (OUT17)
- net G7: now also U4.21 (OUT20)
- net G8: now also U4.24 (OUT23)
- net G9: now also U4.27 (OUT26)
- net GND: now also C3.2, J2.2 (Pin_2), J2.3 (Pin_3), C9.2, R9.1, U4.18 (GND), U4.19 (GND), U4.33 (GND), U4.4 (GND), U4.40 (AD), U4.42 (GND), U4.43 (GND), U4.49 (GND); no longer C3.1
- net I2C_SCL_4: now also U4.46 (SCL)
- net I2C_SDA_4: now also U4.45 (SDA)
- net R1: now also U4.47 (OUT1)
- net R10: now also U4.29 (OUT28)
- net R2: now also U4.2 (OUT4)
- net R3: now also U4.6 (OUT7)
- net R4: now also U4.9 (OUT10)
- net R5: now also U4.12 (OUT13)
- net R6: now also U4.15 (OUT16)
- net R7: now also U4.20 (OUT19)
- net R8: now also U4.23 (OUT22)
- net R9: now also U4.26 (OUT25)
- net at R1.2: now also U4.44 (ISET)
Other:
- moved on the sheet: J4, J5, J7
