File: ControlBreakout.kicad_pcb (KiCad board)
At the start: 2 copper layers, 20 x 54.8 mm, 43 parts, among them J1 Conn_01x12, J2 Conn_01x12, J3 3v3 Bypass, J4 GND1, J5 GND2, J6 Screw_Terminal_01x02, J7 GND3, Q1 AO3401A, U1 TCA9544A, U2 LP5030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

Commit message: nearly done on v2
Parts:
- removed U2: LP5030, Package_DFN_QFN:VQFN-46-1EP_5x6mm_P0.4mm_EP2.8x3.8mm
- added C9: 10uF, Capacitor_SMD:C_0603_1608Metric, F.Cu at (120.6, 108.6)
- added R9: 100K, Resistor_SMD:R_0603_1608Metric, F.Cu at (117.4, 111.8)
- added U4: IS32FL3237-TQLA3-TR, Package_QFP:TQFP-48-1EP_7x7mm_P0.5mm_EP5x5mm, F.Cu at (114.1, 104.6)
- C3, C5: value 1uF -> 100nF; footprint Capacitor_SMD:C_0402_1005Metric -> Capacitor_SMD:C_0603_1608Metric
- C7, C8: footprint Capacitor_SMD:C_0603_1608Metric -> Capacitor_SMD:C_1206_3216Metric
- R1: value 3K -> 3.3K
- moved G*** 144.7 mm to (0.00, 0.00)
- moved C3 11.5 mm to (119.0, 109.5)
- moved R1 6.45 mm to (120.6, 102.4), turned to 90 degrees
- moved C5 6.18 mm to (120.6, 105.5), turned to 90 degrees
- moved R8 3.50 mm to (116.7, 97.3), turned to 0 degrees
- moved D12 3.36 mm to (113.5, 95.8), turned to 180 degrees
- moved J1 2.54 mm to (122.5, 91.3)
- moved R2 2.10 mm to (114.3, 112.9)
- moved U1 2.10 mm to (115.9, 117.2)
- moved C1 2.10 mm to (118.8, 113.1)
- moved C2 2.10 mm to (116.8, 113.1)
- moved C6 1.90 mm to (117.1, 88.0)
- moved D9 1.90 mm to (116.8, 79.0)
- moved F1 1.90 mm to (114.2, 76.9)
- moved FB1 1.90 mm to (117.4, 75.5)
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Connections:
- C3 pad 1: GND -> +3V3
- C3 pad 2: Net-(C3-Pad2) -> GND
- J2 pad 2: +3V3 -> GND
- J2 pad 3: +3V3 -> GND
Routing:
- net GND: track 26.8 -> 93.3 mm, vias 35 -> 193
- net I2C_SCL_4: track 44.2 -> 24.6 mm
- net I2C_SDA_4: track 36.4 -> 22.3 mm
- net B5: track 14.8 -> 2.77 mm, vias 2 -> 0
- net B6: track 14.5 -> 2.93 mm
- net +3V3: track 122.2 -> 133.6 mm
- net R9: track 18.5 -> 7.77 mm, vias 2 -> 0
- net B9: track 19.4 -> 9.90 mm, vias 2 -> 0
- net B10: track 23.9 -> 14.6 mm, vias 2 -> 0
- net G9: track 20.1 -> 10.9 mm, vias 2 -> 0
- net G10: track 24.1 -> 15.1 mm, vias 2 -> 0
- net R6: track 11.3 -> 2.64 mm
- net R10: track 20.6 -> 12.1 mm, vias 2 -> 0
- net B1: track 27.3 -> 19.8 mm
- net G5: track 12.1 -> 4.75 mm, vias 2 -> 0
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Other:
- board size 20 x 54.8 mm -> 20.6 x 54.8 mm

Commit message: First attempt at ordering
Parts:
- moved G*** 143.3 mm to (112.5, 88.8)
